File: hardware/badge-dragonJARCon-2024.kicad_pcb (KiCad board)
At the start: 2 copper layers, 104.7 x 107 mm, 64 parts, among them J1 UART, J2 Battery, J3 OLED, J5 Shitty addon, P1 USB_C_Plug_USB2.0, Q1 DMG3415U-7, SW1 ON, SW2 RESET, SW3 BOOT, SW4 PB4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

Commit message: fix(Hw): update labels
Parts:
- moved kibuzzard-664510D9 4.40 mm to (156.0, 59.2), turned to -160 degrees
- moved kibuzzard-664510CB 4.08 mm to (160.7, 57.5), turned to -160 degrees

Commit message: feat(hw): add labels
Parts:
- moved kibuzzard-66450F45 9.80 mm to (180.2, 31.9)
Other:
- board text added: "America, yo soy... Para los pueblos de América, Les canto mi cancion..."
- board text added: "Sponsored by"
- board text removed: "Parcero usted termina enguayabado"
